Commit message: Fix ur5_robotiq_85.urdf

File: corallab_assets/ur5/ur5_robotiq_85.urdf (robot description, URDF)
Before this commit: robot ur5_robotiq_85, 20 links, 19 joints
Links:
- link base_link: geometry collision mesh filename=./meshes/collision/base.stl; visual mesh filename=./meshes/visual/base.obj
- link forearm_link: geometry collision mesh filename=./meshes/collision/forearm.stl; visual mesh filename=./meshes/visual/forearm.obj
- link left_inner_finger: geometry collision mesh filename=../robotiq_85/meshes/collision/robotiq_arg2f_85_inner_finge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 scale=0.001 0.001 0.001; visual mesh filename=../robotiq_85/meshes/visual/robotiq_arg2f_85_inner_finger.d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 scale=0.001 0.001 0.001
- link left_inner_knuckle: geometry collision mesh filename=../robotiq_85/meshes/collision/robotiq_arg2f_85_inner_knuck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 scale=0.001 0.001 0.001; visual mesh filename=../robotiq_85/meshes/visual/robotiq_arg2f_85_inner_knuckle.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 scale=0.001 0.001 0.001
- link left_outer_finger: geometry collision mesh filename=../robotiq_85/meshes/collision/robotiq_arg2f_85_outer_finge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 scale=0.001 0.001 0.001; visual mesh filename=../robotiq_85/meshes/visual/robotiq_arg2f_85_outer_finger.d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 scale=0.001 0.001 0.001
- link left_outer_knuckle: geometry collision mesh filename=../robotiq_85/meshes/collision/robotiq_arg2f_85_outer_knuck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 scale=0.001 0.001 0.001; visual mesh filename=../robotiq_85/meshes/visual/robotiq_arg2f_85_outer_knuckle.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 scale=0.001 0.001 0.001
- link right_inner_finger: geometry collision mesh filename=../robotiq_85/meshes/collision/robotiq_arg2f_85_inner_finge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 scale=0.001 0.001 0.001; visual mesh filename=../robotiq_85/meshes/visual/robotiq_arg2f_85_inner_finger.d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 scale=0.001 0.001 0.001
- link right_inner_knuckle: geometry collision mesh filename=../robotiq_85/meshes/collision/robotiq_arg2f_85_inner_knuck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 scale=0.001 0.001 0.001; visual mesh filename=../robotiq_85/meshes/visual/robotiq_arg2f_85_inner_knuckle.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 scale=0.001 0.001 0.001
- link right_outer_finger: geometry collision mesh filename=../robotiq_85/meshes/collision/robotiq_arg2f_85_outer_finge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 scale=0.001 0.001 0.001; visual mesh filename=../robotiq_85/meshes/visual/robotiq_arg2f_85_outer_finger.d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 scale=0.001 0.001 0.001
- link right_outer_knuckle: geometry collision mesh filename=../robotiq_85/meshes/collision/robotiq_arg2f_85_outer_knuck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 scale=0.001 0.001 0.001; visual mesh filename=../robotiq_85/meshes/visual/robotiq_arg2f_85_outer_knuckle.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 scale=0.001 0.001 0.001
- link robotiq_arg2f_base_link: geometry collision mesh filename=../robotiq_85/meshes/collision/robotiq_arg2f_base_link.stl; visual mesh filename=../robotiq_85/meshes/visual/robotiq_arg2f_85_base_link.dae scale=0.001 0.001 0.001
- link shoulder_link: geometry collision mesh filename=./meshes/collision/shoulder.stl; visual mesh filename=./meshes/visual/shoulder.obj
- link upper_arm_link: geometry collision mesh filename=./meshes/collision/upperarm.stl; visual mesh filename=./meshes/visual/upperarm.obj
- link wrist_1_link: geometry collision mesh filename=./meshes/collision/wrist1.stl; visual mesh filename=./meshes/visual/wrist1.obj
- link wrist_2_link: geometry collision mesh filename=./meshes/collision/wrist2.stl; visual mesh filename=./meshes/visual/wrist2.obj
- link wrist_3_link: geometry collision mesh filename=./meshes/collision/wrist3.stl; visual mesh filename=./meshes/visual/wrist3.obj
