Commit message: Slightly reformat ur5.urdf

File: corallab_assets/ur5/ur5.urdf (robot description, URDF)
Before this commit: robot ur5, 9 links, 8 joints
Links:
- removed link world
- link base_link: geometry collision mesh filename=meshes/collision/base.stl; visual mesh filename=meshes/visual/base.obj
- link forearm_link: geometry collision mesh filename=meshes/collision/forearm.stl; visual mesh filename=meshes/visual/forearm.obj
- link shoulder_link: geometry collision mesh filename=meshes/collision/shoulder.stl; visual mesh filename=meshes/visual/shoulder.obj
- link upper_arm_link: geometry collision mesh filename=meshes/collision/upperarm.stl; visual mesh filename=meshes/visual/upperarm.obj
- link wrist_1_link: geometry collision mesh filename=meshes/collision/wrist1.stl; visual mesh filename=meshes/visual/wrist1.obj
- link wrist_2_link: geometry collision mesh filename=meshes/collision/wrist2.stl; visual mesh filename=meshes/visual/wrist2.obj
- link wrist_3_link: geometry collision mesh filename=meshes/collision/wrist3.stl; visual mesh filename=meshes/visual/wrist3.obj
Joints:
- removed joint world_arm_joint
