Commit message: Add differently colored cubes

File: corallab_assets/objects/cubes/green_cube.urdf (robot description, URDF)
Before this commit: robot cube, 1 links, 0 joints
Links:
- removed link _name
- added link brown_cube, mass 1.0; collision mesh filename=cube/tinker_vhacd.obj scale=0.001 0.001 0.0009; visual mesh filename=cube/tinker.obj scale=0.001 0.001 0.001
