Commit message: Commit everything

File: corallab_assets/triple_ur5/triple_ur5.urdf (robot description, URDF)
Before this commit: robot dual_ur5_robot, 17 links, 16 joints
Links:
- added link base_link_2, mass 4.0; collision mesh filename=../ur5/meshes/collision/base.stl; visual mesh filename=../ur5/meshes/visual/base.obj
- added link ee_link_2; collision box size=0.01 0.01 0.01
- added link forearm_link_2, mass 2.275; collision mesh filename=../ur5/meshes/collision/forearm.stl; visual mesh filename=../ur5/meshes/visual/forearm.obj
- added link shoulder_link_2, mass 3.7; collision mesh filename=../ur5/meshes/collision/shoulder.stl; visual mesh filename=../ur5/meshes/visual/shoulder.obj
- added link upper_arm_link_2, mass 8.393; collision mesh filename=../ur5/meshes/collision/upperarm.stl; visual mesh filename=../ur5/meshes/visual/upperarm.obj
- added link wrist_1_link_2, mass 1.219; collision mesh filename=../ur5/meshes/collision/wrist1.stl; visual mesh filename=../ur5/meshes/visual/wrist1.obj
- added link wrist_2_link_2, mass 1.219; collision mesh filename=../ur5/meshes/collision/wrist2.stl; visual mesh filename=../ur5/meshes/visual/wrist2.obj
- added link wrist_3_link_2, mass 0.1879; collision mesh filename=../ur5/meshes/collision/wrist3.stl; visual mesh filename=../ur5/meshes/visual/wrist3.obj
- link base_link_0: geometry collision mesh filename=../ur5/meshes/collision/base.stl; visual mesh filename=../ur5/meshes/visual/base.obj
- link base_link_1: geometry collision mesh filename=../ur5/meshes/collision/base.stl; visual mesh filename=../ur5/meshes/visual/base.obj
- link forearm_link_0: geometry collision mesh filename=../ur5/meshes/collision/forearm.stl; visual mesh filename=../ur5/meshes/visual/forearm.obj
- link forearm_link_1: geometry collision mesh filename=../ur5/meshes/collision/forearm.stl; visual mesh filename=../ur5/meshes/visual/forearm.obj
- link shoulder_link_0: geometry collision mesh filename=../ur5/meshes/collision/shoulder.stl; visual mesh filename=../ur5/meshes/visual/shoulder.obj
- link shoulder_link_1: geometry collision mesh filename=../ur5/meshes/collision/shoulder.stl; visual mesh filename=../ur5/meshes/visual/shoulder.obj
- link upper_arm_link_0: geometry collision mesh filename=../ur5/meshes/collision/upperarm.stl; visual mesh filename=../ur5/meshes/visual/upperarm.obj
- link upper_arm_link_1: geometry collision mesh filename=../ur5/meshes/collision/upperarm.stl; visual mesh filename=../ur5/meshes/visual/upperarm.obj
- link wrist_1_link_0: geometry collision mesh filename=../ur5/meshes/collision/wrist1.stl; visual mesh filename=../ur5/meshes/visual/wrist1.obj
- link wrist_1_link_1: geometry collision mesh filename=../ur5/meshes/collision/wrist1.stl; visual mesh filename=../ur5/meshes/visual/wrist1.obj
- link wrist_2_link_0: geometry collision mesh filename=../ur5/meshes/collision/wrist2.stl; visual mesh filename=../ur5/meshes/visual/wrist2.obj
- link wrist_2_link_1: geometry collision mesh filename=../ur5/meshes/collision/wrist2.stl; visual mesh filename=../ur5/meshes/visual/wrist2.obj
- link wrist_3_link_0: geometry collision mesh filename=../ur5/meshes/collision/wrist3.stl; visual mesh filename=../ur5/meshes/visual/wrist3.obj
- link wrist_3_link_1: geometry collision mesh filename=../ur5/meshes/collision/wrist3.stl; visual mesh filename=../ur5/meshes/visual/wrist3.obj
Joints:
- added joint base_link_joint_2: type fixed, parent base_fixture_link, child base_link_2, origin xyz=0.50 -0.25 0.1 rpy=0 0 3.1415
- added joint ee_fixed_joint_2: type fixed, parent wrist_3_link_2, child ee_link_2, origin xyz=0.0 0.0823 0.0 rpy=0.0 0.0 1.57079632679
- added joint elbow_joint_2: type revolute, parent upper_arm_link_2, child forearm_link_2, origin xyz=0.0 -0.1197 0.425 rpy=0.0 0.0 0.0, axis 0 1 0, limit lower=-3.14159265359 upper=3.14159265359 effort=150.0 velocity=3.15
- added joint shoulder_lift_joint_2: type revolute, parent shoulder_link_2, child upper_arm_link_2, origin xyz=0.0 0.13585 0.0 rpy=0.0 1.57079632679 0.0, axis 0 1 0, limit lower=-3.14159265359 upper=3.14159265359 effort=150.0 velocity=3.15
- added joint shoulder_pan_joint_2: type revolute, parent base_link_2, child shoulder_link_2, origin xyz=0.0 0.0 0.089159 rpy=0.0 0.0 0.0, axis 0 0 1, limit lower=-3.14159265359 upper=3.14159265359 effort=150.0 velocity=3.15
- added joint wrist_1_joint_2: type revolute, parent forearm_link_2, child wrist_1_link_2, origin xyz=0.0 0.0 0.39225 rpy=0.0 1.57079632679 0.0, axis 0 1 0, limit lower=-3.14159265359 upper=3.14159265359 effort=28.0 velocity=3.2
- added joint wrist_2_joint_2: type revolute, parent wrist_1_link_2, child wrist_2_link_2, origin xyz=0.0 0.093 0.0 rpy=0.0 0.0 0.0, axis 0 0 1, limit lower=-3.14159265359 upper=3.14159265359 effort=28.0 velocity=3.2
- added joint wrist_3_joint_2: type revolute, parent wrist_2_link_2, child wrist_3_link_2, origin xyz=0.0 0.0 0.09465 rpy=0.0 0.0 0.0, axis 0 1 0, limit lower=-3.14159265359 upper=3.14159265359 effort=28.0 velocity=3.2
- joint base_link_joint_0: origin xyz=0.50 0.0 0.1 rpy=0 0 3.1415 -> xyz=0.50 0.25 0.1 rpy=0 0 3.1415
- joint wrist_3_joint_0: limit lower=-6.28318530718 upper=6.28318530718 effort=28.0 velocity=3.2 -> lower=-3.14159265359 upper=3.14159265359 effort=28.0 velocity=3.2
- joint wrist_3_joint_1: limit lower=-6.28318530718 upper=6.28318530718 effort=28.0 velocity=3.2 -> lower=-3.14159265359 upper=3.14159265359 effort=28.0 velocity=3.2

File: corallab_assets/triple_ur5/triple_ur5_test.urdf (robot description, URDF)
Before this commit: robot dual_ur5_robot, 17 links, 16 joints
Links:
- added link base_link_2, mass 4.0; collision mesh filename=../ur5/meshes/visual/base.obj; visual mesh filename=../ur5/meshes/visual/base.obj
- added link ee_link_2; collision box size=0.01 0.01 0.01
- added link forearm_link_2, mass 2.275; collision mesh filename=../ur5/meshes/visual/forearm.obj; visual mesh filename=../ur5/meshes/visual/forearm.obj
- added link shoulder_link_2, mass 3.7; collision mesh filename=../ur5/meshes/visual/shoulder.obj; visual mesh filename=../ur5/meshes/visual/shoulder.obj
- added link upper_arm_link_2, mass 8.393; collision mesh filename=../ur5/meshes/visual/upperarm.obj; visual mesh filename=../ur5/meshes/visual/upperarm.obj
- added link wrist_1_link_2, mass 1.219; collision mesh filename=../ur5/meshes/visual/wrist1.obj; visual mesh filename=../ur5/meshes/visual/wrist1.obj
- added link wrist_2_link_2, mass 1.219; collision mesh filename=../ur5/meshes/visual/wrist2.obj; visual mesh filename=../ur5/meshes/visual/wrist2.obj
- added link wrist_3_link_2, mass 0.1879; collision mesh filename=../ur5/meshes/visual/wrist3.obj; visual mesh filename=../ur5/meshes/visual/wrist3.obj
- link base_link_0: geometry collision mesh filename=../ur5/meshes/visual/base.obj; visual mesh filename=../ur5/meshes/visual/base.obj
- link base_link_1: geometry collision mesh filename=../ur5/meshes/visual/base.obj; visual mesh filename=../ur5/meshes/visual/base.obj
- link forearm_link_0: geometry collision mesh filename=../ur5/meshes/visual/forearm.obj; visual mesh filename=../ur5/meshes/visual/forearm.obj
- link forearm_link_1: geometry collision mesh filename=../ur5/meshes/visual/forearm.obj; visual mesh filename=../ur5/meshes/visual/forearm.obj
- link shoulder_link_0: geometry collision mesh filename=../ur5/meshes/visual/shoulder.obj; visual mesh filename=../ur5/meshes/visual/shoulder.obj
- link shoulder_link_1: geometry collision mesh filename=../ur5/meshes/visual/shoulder.obj; visual mesh filename=../ur5/meshes/visual/shoulder.obj
- link upper_arm_link_0: geometry collision mesh filename=../ur5/meshes/visual/upperarm.obj; visual mesh filename=../ur5/meshes/visual/upperarm.obj
- link upper_arm_link_1: geometry collision mesh filename=../ur5/meshes/visual/upperarm.obj; visual mesh filename=../ur5/meshes/visual/upperarm.obj
- link wrist_1_link_0: geometry collision mesh filename=../ur5/meshes/visual/wrist1.obj; visual mesh filename=../ur5/meshes/visual/wrist1.obj
- link wrist_1_link_1: geometry collision mesh filename=../ur5/meshes/visual/wrist1.obj; visual mesh filename=../ur5/meshes/visual/wrist1.obj
- link wrist_2_link_0: geometry collision mesh filename=../ur5/meshes/visual/wrist2.obj; visual mesh filename=../ur5/meshes/visual/wrist2.obj
- link wrist_2_link_1: geometry collision mesh filename=../ur5/meshes/visual/wrist2.obj; visual mesh filename=../ur5/meshes/visual/wrist2.obj
- link wrist_3_link_0: geometry collision mesh filename=../ur5/meshes/visual/wrist3.obj; visual mesh filename=../ur5/meshes/visual/wrist3.obj
- link wrist_3_link_1: geometry collision mesh filename=../ur5/meshes/visual/wrist3.obj; visual mesh filename=../ur5/meshes/visual/wrist3.obj
Joints:
- added joint base_link_joint_2: type fixed, parent base_fixture_link, child base_link_2, origin xyz=0.50 -0.25 0.1 rpy=0 0 3.1415
- added joint ee_fixed_joint_2: type fixed, parent wrist_3_link_2, child ee_link_2, origin xyz=0.0 0.0823 0.0 rpy=0.0 0.0 1.57079632679
- added joint elbow_joint_2: type revolute, parent upper_arm_link_2, child forearm_link_2, origin xyz=0.0 -0.1197 0.425 rpy=0.0 0.0 0.0, axis 0 1 0, limit lower=-3.14159265359 upper=3.14159265359 effort=150.0 velocity=3.15
- added joint shoulder_lift_joint_2: type revolute, parent shoulder_link_2, child upper_arm_link_2, origin xyz=0.0 0.13585 0.0 rpy=0.0 1.57079632679 0.0, axis 0 1 0, limit lower=-3.14159265359 upper=3.14159265359 effort=150.0 velocity=3.15
- added joint shoulder_pan_joint_2: type revolute, parent base_link_2, child shoulder_link_2, origin xyz=0.0 0.0 0.089159 rpy=0.0 0.0 0.0, axis 0 0 1, limit lower=-3.14159265359 upper=3.14159265359 effort=150.0 velocity=3.15
- added joint wrist_1_joint_2: type revolute, parent forearm_link_2, child wrist_1_link_2, origin xyz=0.0 0.0 0.39225 rpy=0.0 1.57079632679 0.0, axis 0 1 0, limit lower=-3.14159265359 upper=3.14159265359 effort=28.0 velocity=3.2
- added joint wrist_2_joint_2: type revolute, parent wrist_1_link_2, child wrist_2_link_2, origin xyz=0.0 0.093 0.0 rpy=0.0 0.0 0.0, axis 0 0 1, limit lower=-3.14159265359 upper=3.14159265359 effort=28.0 velocity=3.2
- added joint wrist_3_joint_2: type revolute, parent wrist_2_link_2, child wrist_3_link_2, origin xyz=0.0 0.0 0.09465 rpy=0.0 0.0 0.0, axis 0 1 0, limit lower=-3.14159265359 upper=3.14159265359 effort=28.0 velocity=3.2
- joint base_link_joint_0: origin xyz=0.50 0.0 0.1 rpy=0 0 3.1415 -> xyz=0.50 0.25 0.1 rpy=0 0 3.1415
- joint wrist_3_joint_0: limit lower=-6.28318530718 upper=6.28318530718 effort=28.0 velocity=3.2 -> lower=-3.14159265359 upper=3.14159265359 effort=28.0 velocity=3.2
- joint wrist_3_joint_1: limit lower=-6.28318530718 upper=6.28318530718 effort=28.0 velocity=3.2 -> lower=-3.14159265359 upper=3.14159265359 effort=28.0 velocity=3.2

File: corallab_assets/ur5/ur5_test.urdf (robot description, URDF)
Before this commit: robot ur5, 9 links, 8 joints
Links:
- link base_link: geometry collision mesh filename=meshes/visual/base.obj; visual mesh filename=meshes/visual/base.obj
- link forearm_link: geometry collision mesh filename=meshes/visual/forearm.obj; visual mesh filename=meshes/visual/forearm.obj
- link shoulder_link: geometry collision mesh filename=meshes/visual/shoulder.obj; visual mesh filename=meshes/visual/shoulder.obj
- link upper_arm_link: geometry collision mesh filename=meshes/visual/upperarm.obj; visual mesh filename=meshes/visual/upperarm.obj
- link wrist_1_link: geometry collision mesh filename=meshes/visual/wrist1.obj; visual mesh filename=meshes/visual/wrist1.obj
- link wrist_2_link: geometry collision mesh filename=meshes/visual/wrist2.obj; visual mesh filename=meshes/visual/wrist2.obj
- link wrist_3_link: geometry collision mesh filename=meshes/visual/wrist3.obj; visual mesh filename=meshes/visual/wrist3.obj
